File: pcb/Tesla Ambient Lighting.kicad_sch (KiCad schematic)
At the start: 21 parts, among them J1 LED_1, J2 LED_2, J3 LED_3, J4 LED_4, J5 CHASSIS_CAN, J6 USB4105-GF-A, J7 Screw_Terminal_01x02, SW1 BOOT_OPTION, U1 ESP32-WROOM-32, U2 SN65HVD230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

Commit message: started PCB V2; adding DTR and RTS control pins, RST button, and power LED; also wanting to add serial LED
Parts:
- added D1: PWR_LED, LED_SMD:LED_0805_2012Metric, symbol Device:LED
- added Q1, Q2: Q_NPN_BEC, Package_TO_SOT_SMD:SOT-23, symbol Transistor_BJT:Q_NPN_BEC
- added R6: 50, Resistor_SMD:R_0805_2012Metric, symbol Device:R
- added R7, R8, R9: 10k, Resistor_SMD:R_0805_2012Metric, symbol Device:R
- added SW2: RESET, Button_Switch_SMD:SW_SPST_B3U-1100P, symbol Switch:SW_Push
Connections:
- net GNDREF: now also U5.1 (~{DTR}), D1.1 (K), Q2.2 (E), R8.1, SW2.1
- net V33: now also R6.1
- net V5: now also R7.1
- net GPIO0: now reaches SW1.1, U1.25 (IO0)
- net GPIO0: now also Q2.3 (C), R7.2
- net EN: now reaches C3.2, R1.2, U1.3 (EN)
- net EN: now also Q1.3 (C), SW2.2
- net RTS: now reaches U5.2 (~{RTS})
- net RTS: now also Q1.2 (E), R9.1
- new net: D1.2 (A), R6.2
- new net: Q2.1 (B), R9.2
- new net: Q1.1 (B), R8.2
- no-connect marks 36 -> 34
Other:
- moved on the sheet: C3, R1, U1, U2
